Commit message: cpp version

File: test/test.urdf (robot description, URDF)
Before this commit: robot testboii, 2 links, 1 joints
Links:
- removed link first
- removed link second
- added link base_link; collision mesh filename=package://wolfgang_description/urdf/nuc_holder_left_back.stl; visual mesh filename=package://wolfgang_description/urdf/nuc_holder_left_back.stl
Joints:
- removed joint blub

File: test/wolfgang_boxed.urdf (robot description, URDF)
Before this commit: robot wolfgang, 48 links, 47 joints
Links:
- link head: geometry collision box size=0.004499999806284913 0.06117891295941271 0.0611789129594127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; collision box size=0.007094643311575065 0.058097971880820366 0.128278347570678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
- link l_ankle: geometry collision box size=0.005599999800334421 0.029999999329447746 0.030999999493360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; collision box size=0.006000000052154064 0.011599999852478506 0.028000000864267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
- link l_foot: geometry collision box size=0.0015999999595806113 0.05999999865889549 0.0599999986588955; collision box size=0.004000000189989805 0.008000000379979616 0.039999999105930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
- link l_hip_1: geometry collision box size=0.05000000167638064 0.053174532949924476 0.10000000149011612; visual mesh filename=package://wolfgang_description/urdf/l_hip_1.stl
- link l_hip_2: geometry collision box size=0.005599999800334421 0.029999999329447746 0.030999999493360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; collision box size=0.006000000052154064 0.011599999852478506 0.028000000864267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
- link l_lower_arm: geometry collision box size=0.0020000000949949026 0.07899051974556984 0.232322900889016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; collision box size=0.0020000000949949026 0.07899051974556984 0.232322900889016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
- link l_lower_leg: geometry collision box size=0.0015000011771917373 0.03596901059332641 0.035975066861305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; collision box size=0.0015000011771917373 0.03596901059332641 0.035975066861305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
- link l_shoulder: geometry collision box size=0.004499999806284913 0.06117891295941271 0.0611789129594127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; collision box size=0.008999999612569818 0.04995241066301348 0.04995241066301346
- link l_upper_arm: geometry collision box size=0.0022499999322462827 0.03999999910593034 0.170000005513429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; collision box size=0.0022499999322462827 0.03999999910593034 0.170000005513429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
- link l_upper_leg: geometry collision box size=0.002000000094994907 0.05203729183943207 0.1715830404353845; collision box size=0.002000000094994907 0.05203729183943207 0.1715830404353845
- link llb: geometry collision box size=0.012987822030476881 0.012987822030476886 0.015999999828636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; visual mesh filename=package://wolfgang_description/urdf/llb.stl
- link llf: geometry collision box size=0.012987822030476881 0.012987822030476886 0.015999999828636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; visual mesh filename=package://wolfgang_description/urdf/llf.stl
- link lrb: geometry collision box size=0.012987822030476881 0.012987822030476886 0.015999999828636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; visual mesh filename=package://wolfgang_description/urdf/lrb.stl
- link lrf: geometry collision box size=0.012987822030476881 0.012987822030476886 0.015999999828636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; visual mesh filename=package://wolfgang_description/urdf/lrf.stl
- link neck: geometry collision box size=0.009300000034272672 0.035999998450279236 0.039999999105930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; collision box size=0.04019999876618386 0.04609999991953373 0.061099998652935035
- link r_ankle: geometry collision box size=0.005599999800334421 0.029999999329447746 0.030999999493360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; collision box size=0.006000000052154064 0.011599999852478506 0.028000000864267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
- link r_foot: geometry collision box size=0.0015999999595806113 0.05999999865889549 0.0599999986588955; collision box size=0.004000000189989805 0.008000000379979616 0.039999999105930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
- link r_hip_1: geometry collision box size=0.05000000167638064 0.053174532949924476 0.10000000149011612; visual mesh filename=package://wolfgang_description/urdf/r_hip_1.stl
- link r_hip_2: geometry collision box size=0.005599999800334421 0.029999999329447746 0.030999999493360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; collision box size=0.006000000052154064 0.011599999852478506 0.028000000864267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
- link r_lower_arm: geometry collision box size=0.0020000000949949026 0.07899051974556984 0.232322900889016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; collision box size=0.0020000000949949026 0.07899051974556984 0.232322900889016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
- link r_lower_leg: geometry collision box size=0.0015000011771917373 0.03596901059332641 0.035975066861305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; collision box size=0.0015000011771917373 0.03596901059332641 0.035975066861305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
- link r_shoulder: geometry collision box size=0.004499999806284913 0.06117891295941271 0.0611789129594127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; collision box size=0.008999999612569818 0.04995241066301348 0.04995241066301346
- link r_upper_arm: geometry collision box size=0.0022499999322462827 0.03999999910593034 0.170000005513429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; collision box size=0.0022499999322462827 0.03999999910593034 0.170000005513429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
- link r_upper_leg: geometry collision box size=0.002000000094994907 0.05203729183943207 0.1715830404353845; collision box size=0.002000000094994907 0.05203729183943207 0.1715830404353845
- link rlb: geometry collision box size=0.012987822030476881 0.012987822030476886 0.015999999828636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; visual mesh filename=package://wolfgang_description/urdf/rlb.stl
- link rlf: geometry collision box size=0.012987822030476881 0.012987822030476886 0.015999999828636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; visual mesh filename=package://wolfgang_description/urdf/rlf.stl
- link rrb: geometry collision box size=0.012987822030476881 0.012987822030476886 0.015999999828636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; visual mesh filename=package://wolfgang_description/urdf/rrb.stl
- link rrf: geometry collision box size=0.012987822030476881 0.012987822030476886 0.015999999828636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; visual mesh filename=package://wolfgang_description/urdf/rrf.stl
- link torso: geometry collision box size=0.0020000000949949148 0.06599999964237213 0.131999999284744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; collision box size=0.002000000327825547 0.018999999389052395 0.083999998867511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
